File: electrical/USB-PD-Breakout.kicad_pcb (KiCad board)
At the start: 2 copper layers, 34.5 x 28 mm, 25 parts, among them J1 USB-C_Female, J2 USB_OTG, J3 CONN_02X03, J4 Conn_01x08_Male, U1 FUSB302BMPX, X1 MTHOLE, X2 MTHOLE

Commit message: Add SBU header for Apple M1 debug UART
Signed-off-by: Rouven Czerwinski <rouven@czerwinskis.de>
Parts:
- added J5: 640456-3, digikey-footprints:PinHeader_1x3_P2.54_Drill1.1mm, F.Cu at (129.2, 75.5)
- moved TP2 1.99 mm to (127.1, 79.1)
Routing:
- net Net-(J1-PadA8): track 0.00 -> 43.3 mm, vias 0 -> 1
- net Net-(J1-PadB8): track 0.00 -> 38.6 mm, vias 0 -> 1
- net VBUS_A: track 26.6 -> 28.2 mm
- net V_PULLUP: track 16.3 -> 17.7 mm
Other:
- board text added: "SBU1"
- board text added: "SBU1/2"
- board text added: "SBU2"
- board text added: "USB PowerDelivery Breakout Board Rev 4 ReclaimerLabs.com SBU Variant"
- board text removed: "USB PowerDelivery Breakout Board Rev 4 ReclaimerLabs.com"
