File: electrical/USB-PD-Breakout.sch (KiCad schematic (older format))
At the start: 25 parts, among them J1 USB-C_Female, J2 USB_OTG, J3 CONN_02X03, J4 Conn_01x08_Male, U1 FUSB302BMPX, X1 MTHOLE, X2 MTHOLE

Commit message: Add SBU header for Apple M1 debug UART
Signed-off-by: Rouven Czerwinski <rouven@czerwinskis.de>
Parts:
- added J5: 640456-3, digikey-footprints:PinHeader_1x3_P2.54_Drill1.1mm, symbol dk_Rectangular-Connectors-Headers-Male-Pins:640456-3
- C1, C2, C3, C4, C5, C6: symbol Device:C -> USB-PD-Breakout-rescue:C-Device
- J1: symbol Jason_Custom_Home:USB-C_Female -> USB-PD-Breakout-rescue:USB-C_Female-Jason_Custom_Home
- J4: symbol conn:Conn_01x08_Male -> USB-PD-Breakout-rescue:Conn_01x08_Male-conn
- R1, R2, R3: symbol Device:R -> USB-PD-Breakout-rescue:R-Device
- TP1: symbol conn:TEST_1P -> USB-PD-Breakout-rescue:TEST_1P-conn
- TP2, TP3, TP4, TP5, TP6, TP7, TP8, TP9: renamed from TP?; symbol conn:TEST_1P -> USB-PD-Breakout-rescue:TEST_1P-conn
- U1: symbol Jason_Custom_Home:FUSB302MPX -> USB-PD-Breakout-rescue:FUSB302MPX-Jason_Custom_Home
- X1, X2: symbol Jason_Custom_Home:MTHOLE -> USB-PD-Breakout-rescue:MTHOLE-Jason_Custom_Home
Connections:
- net labels added: GND-power
- wire segments 122 -> 129
- no-connect marks 13 -> 12
